Commit message: Model not spawning, URDF deprecation amended

File: ROSject_2/src/mybot_description/urdf/mybot_TEST.xacro (robot description, xacro)
@@ -18,12 +18,7 @@
 	<xacro:property name="cameraSize" value="0.05"/>
 	<xacro:property name="cameraMass" value="0.1"/>
-	<link name="footprint">
-	<joint name="base_joint" type="fixed">
-		<parent link="footprint"/>
-		<child link="chassis"/>
-	</joint>
-	</link>
 	<link name='chassis'>
-		<collision>
+		<pose>0 0 0.1 0 0 0</pose>
+		<collision name="boxCollision">
 			<origin xyz="0 0 ${wheelRadius}" rpy="0 0 0"/>
 			<geometry>
@@ -31,5 +26,21 @@
 			</geometry>
 		</collision>
-		<visual>
+		<collision name="casterCollision">
+			<origin xyz="-0.15 0 -0.05" rpy=" 0 0 0"/>
+			<geometry>
+				<sphere radius="${casterRadius}"/>
+			</geometry>
+			<surface>
+				<friction>
+					<ode>
+						<mu>0</mu>
+						<mu2>0</mu2>
+						<slip1>1.0</slip1>
+						<slip2>1.0</slip2>
+					</ode>
+				</friction>
+			</surface>
+		</collision>
+		<visual name ="chassisVisual">
 			<origin xyz="0 0 ${wheelRadius}" rpy="0 0 0"/>
 			<geometry>
@@ -37,4 +48,10 @@
 			</geometry>
 			<material name="orange"/>
+		</visual>
+		<visual name="casterVisual">
+			origin xyz="-0.15 0 -0.05" rpy=" 0 0 0"/>
+			<geometry>
+				<sphere radius="${casterRadius}"/>
+			</geometry>
 		</visual>
 		<inertial>
@@ -44,3 +61,59 @@
 		</inertial>
 	</link>
+	<link name="left_wheel">
+		<!--origin xyz="0.1 0.13 0.1" rpy="0 1.5707 1.5707"/-->
+		<collision name="collisionLWheel">
+			<origin xyz="0 0 0" rpy="0 1.5707 1.5707"/>
+			<geometry>
+				<cylinder radius="${wheelRadius}" length="{wheelWidth}"/>
+			</geometry>
+		</collision>
+		<visual name="visualLWheel">
+			<origin xyz="0 0 0" rpy="0 1.5707 1.5707"/>
+			<geometry>
+				<cylinder radius="${wheelRadius}" length="{wheelWidth}"/>
+			</geometry>
+		</visual>
+		<inertial>
+			<origin xyz="0 0 0" rpy="0 1.5707 1.5707"/>
+			<mass value="${wheelMass}"/>
+			<cylinder_inertia m="{wheelMass}" r="${wheelRadius}" h="${wheelWidth}"/>
+		</inertial>
+	</link>
+	<link name="right_wheel">
+		<!--origin xyz="0.1 -0.13 0.1" rpy="0 1.5707 1.5707"/-->
+		<collision name="collisionRWheel">
+			<origin xyz="0 0 0" rpy="0 1.5707 1.5707"/>
+			<geometry>
+				<cylinder radius="${wheelRadius}" length="{wheelWidth}"/>
+			</geometry>
+		</collision>
+		<visual name="visualRWheel">
+			<origin xyz="0 0 0" rpy="0 1.5707 1.5707"/>
+			<geometry>
+				<cylinder radius="${wheelRadius}" length="{wheelWidth}"/>
+			</geometry>
+		</visual>
+		<inertial>
+			<origin xyz="0 0 0" rpy="0 1.5707 1.5707"/>
+			<mass value="${wheelMass}"/>
+			<cylinder_inertia m="{wheelMass}" r="${wheelRadius}" h="${wheelWidth}"/>
+		</inertial>
+	</link>
+	<joint type="continuous" name="left_wheel_hinge">
+		<origin xyz="0.1 0.15 0" rpy="0 0 0"/>
+		<child link="left_wheel"/>
+		<parent link="chassis"/>
+		<axis xyz="0 1 0" rpy="0 0 0"/>
+		<limit effort="100" velocity="100"/>
+		<joint_properties damping="0.0" friction="0.0"/>
+	</joint>
+	<joint type="continuous" name="right_wheel_hinge">
+		<origin xyz="0.1 -0.15 0" rpy="0 0 0"/>
+		<child link="right_wheel"/>
+		<parent link="chassis"/>
+		<axis xyz="0 1 0" rpy="0 0 0"/>
+		<limit effort="100" velocity="100"/>
+		<joint_properties damping="0.0" friction="0.0"/>
+	</joint>
 </robot>
