Commit message: **Controller Spawn Working**
Changelog added to mybot_control.launch to remove 'unable to parse URDF' error
L-R Wheel axis rotated by pi. Will need debugging
Simulation colors except chassis generating

File: ROSject_2/src/mybot_description/urdf/materials.xacro (robot description, xacro)
@@ -4,13 +4,13 @@
 	<color rgba="0.0 0.0 0.0 1.0"/>
 </material>
-<material name="blue">
-<color rgba="0.0 0.0 0.8 1.0"/>
-</material>
-<material name="green">
-<color rgba="0.0 0.8 0.0 1.0"/>
-</material>
-<material name="grey">
-<color rgba="0.2 0.2 0.2 1.0"/>
-</material>
+	<material name="blue">
+		<color rgba="0.0 0.0 0.8 1.0"/>
+	</material>
+	<material name="green">
+		<color rgba="0.0 0.8 0.0 1.0"/>
+	</material>
+	<material name="grey">
+		<color rgba="0.2 0.2 0.2 1.0"/>
+	</material>
 	<material name="orange">
 		<color rgba="0.8 0.4 0.0 1.0"/>
@@ -22,6 +22,6 @@
 		<color rgba="0.8 0.0 0.0 1.0"/>
 	</material>
-<material name="white">
-<color rgba="1.0 1.0 1.0 1.0"/>
-</material>
+	<material name="white">
+		<color rgba="1.0 1.0 1.0 1.0"/>
+	</material>
 </robot>

File: ROSject_2/src/mybot_description/urdf/mybot.xacro (robot description, xacro)
@@ -19,17 +19,18 @@
 	<xacro:property name="cameraMass" value="0.1"/>
 	<!-- End of common prperties description -->
-	<link name="footprint">
-	<inertial>
-		<inertia name="baseFrameInertia">
-			ixx="0.0" ixy="0.0" ixz="0.0"
-			iyy="0.0" iyz="0.0"
-			izz="0.0"/>
-		</inertia>
-	</inertial>
-	</link>
-	<joint name="base_joint" type="fixed">
-		<parent link="footprint"/>
-		<child link="chassis"/>
-	</joint>
+<!--	<link name="footprint">-->
+<!--	<inertial>-->
+<!--		<mass value="0.0"/>-->
+<!--		<inertia name="baseFrameInertia">-->
+<!--			ixx="1.0" ixy="0.0" ixz="0.0"-->
+<!--			iyy="0.0" iyz="0.0"-->
+<!--			izz="0.0"/>-->
+<!--		</inertia>-->
+<!--	</inertial>-->
+<!--	</link>-->
+<!--	<joint name="base_joint" type="fixed">-->
+<!--		<parent link="footprint"/>-->
+<!--		<child link="chassis"/>-->
+<!--	</joint>-->
 	<link name='chassis'>
 		<pose>0 0 0.1 0 0 0</pose>
@@ -78,4 +79,5 @@
 		</inertial>
 	</link>
+<!--Macros for wheels: Links and Joints both-->
 	<xacro:wheel lr="left" tY="1"/>
 	<xacro:wheel lr="right" tY="-1"/>
