Commit message: Macros working, URDF deprecation issue unresolved

File: ROSject_2/src/mybot_description/urdf/macros.xacro (robot description, xacro)
@@ -1,69 +1,69 @@
 <?xml version="1.0"?>
-<robot>
-	<macro name="cylinder_inertia" params="m r h">
+<robot xmlns:xacro="http://www.ros.org/wiki/xacro"> <!-- NAMESPACE WAS MISSING, USE xacro:macro instead of just macro -->
+	<xacro:macro name="cylinder_inertia" params="m r h">
 	  <inertia  ixx="${m*(3*r*r+h*h)/12}" ixy = "0" ixz = "0"
 		iyy="${m*(3*r*r+h*h)/12}" iyz = "0"
 		izz="${m*r*r/2}"
 	  />
-	</macro>
-	<macro name="box_inertia" params="m x y z">
+	</xacro:macro>
+	<xacro:macro name="box_inertia" params="m x y z">
 	  <inertia  ixx="${m*(y*y+z*z)/12}" ixy = "0" ixz = "0"
 		iyy="${m*(x*x+z*z)/12}" iyz = "0"
 		izz="${m*(x*x+z*z)/12}"
 	  />
-	</macro>
-	<macro name="sphere_inertia" params="m r">
+	</xacro:macro>
+	<xacro:macro name="sphere_inertia" params="m r">
 	  <inertia  ixx="${2*m*r*r/5}" ixy = "0" ixz = "0"
 		iyy="${2*m*r*r/5}" iyz = "0"
 		izz="${2*m*r*r/5}"
 	  />
-	</macro>
-	<macro name="wheel" params="lr tY">
-	  <link name="${lr}_wheel">
-		<collision>
-		  <origin xyz="0 0 0" rpy="0 ${PI/2} ${PI/2}" />
-		  <geometry>
-			<cylinder length="${wheelWidth}" radius="${wheelRadius}"/>
-		  </geometry>
-		</collision>
-		<visual>
-		  <origin xyz="0 0 0" rpy="0 ${PI/2} ${PI/2}" />
-		  <geometry>
-			<cylinder length="${wheelWidth}" radius="${wheelRadius}"/>
-		  </geometry>
-		  <material name="black"/>
-		</visual>
-		<inertial>
-		  <origin xyz="0 0 0" rpy="0 ${PI/2} ${PI/2}" />
-		  <mass value="${wheelMass}"/>
-		  <cylinder_inertia m="${wheelMass}" r="${wheelRadius}" h="${wheelWidth}"/>
-		</inertial>
-	  </link>
-	  <gazebo reference="${lr}_wheel">
-		<mu1 value="1.0"/>
-		<mu2 value="1.0"/>
-		<kp  value="10000000.0" />
-		<kd  value="1.0" />
-		<fdir1 value="1 0 0"/>
-		<material>Gazebo/Black</material>
-	  </gazebo>
-	  <joint name="${lr}_wheel_hinge" type="continuous">
-		<parent link="chassis"/>
-		<child link="${lr}_wheel"/>
-	  <origin xyz="${-wheelPos+chassisLength/2} ${tY*wheelWidth/2+tY*chassisWidth/2} ${wheelRadius}" rpy="0 0 0" />
-		<axis xyz="0 1 0" rpy="0 0 0" />
-		<limit effort="10000" velocity="10000"/>
-		<joint_properties damping="0.0" friction="0.0"/>
-	  </joint>
-	  <transmission name="${lr}_trans">
-		<type>transmission_interface/SimpleTransmission</type>
-		<joint name="${lr}_wheel_hinge">
-		  <hardwareInterface>EffortJointInterface</hardwareInterface>
-		</joint>
-		<actuator name="${lr}Motor">
-		  <hardwareInterface>EffortJointInterface</hardwareInterface>
-		  <mechanicalReduction>10</mechanicalReduction>
-		</actuator>
-	  </transmission>
-	</macro>
+	</xacro:macro>
+<!--	<macro name="wheel" params="lr tY">-->
+<!--	  <link name="${lr}_wheel">-->
+<!--		<collision>-->
+<!--		  <origin xyz="0 0 0" rpy="0 ${PI/2} ${PI/2}" />-->
+<!--		  <geometry>-->
+<!--			<cylinder length="${wheelWidth}" radius="${wheelRadius}"/>-->
+<!--		  </geometry>-->
+<!--		</collision>-->
+<!--		<visual>-->
+<!--		  <origin xyz="0 0 0" rpy="0 ${PI/2} ${PI/2}" />-->
+<!--		  <geometry>-->
+<!--			<cylinder length="${wheelWidth}" radius="${wheelRadius}"/>-->
+<!--		  </geometry>-->
+<!--		  <material name="black"/>-->
+<!--		</visual>-->
+<!--		<inertial>-->
+<!--		  <origin xyz="0 0 0" rpy="0 ${PI/2} ${PI/2}" />-->
+<!--		  <mass value="${wheelMass}"/>-->
+<!--		  <cylinder_inertia m="${wheelMass}" r="${wheelRadius}" h="${wheelWidth}"/>-->
+<!--		</inertial>-->
+<!--	  </link>-->
+<!--	  <gazebo reference="${lr}_wheel">-->
+<!--		<mu1 value="1.0"/>-->
+<!--		<mu2 value="1.0"/>-->
+<!--		<kp  value="10000000.0" />-->
+<!--		<kd  value="1.0" />-->
+<!--		<fdir1 value="1 0 0"/>-->
+<!--		<material>Gazebo/Black</material>-->
+<!--	  </gazebo>-->
+<!--	  <joint name="${lr}_wheel_hinge" type="continuous">-->
+<!--		<parent link="chassis"/>-->
+<!--		<child link="${lr}_wheel"/>-->
+<!--	  <origin xyz="${-wheelPos+chassisLength/2} ${tY*wheelWidth/2+tY*chassisWidth/2} ${wheelRadius}" rpy="0 0 0" />-->
+<!--		<axis xyz="0 1 0" rpy="0 0 0" />-->
+<!--		<limit effort="10000" velocity="10000"/>-->
+<!--		<joint_properties damping="0.0" friction="0.0"/>-->
+<!--	  </joint>-->
+<!--	  <transmission name="${lr}_trans">-->
+<!--		<type>transmission_interface/SimpleTransmission</type>-->
+<!--		<joint name="${lr}_wheel_hinge">-->
+<!--		  <hardwareInterface>EffortJointInterface</hardwareInterface>-->
+<!--		</joint>-->
+<!--		<actuator name="${lr}Motor">-->
+<!--		  <hardwareInterface>EffortJointInterface</hardwareInterface>-->
+<!--		  <mechanicalReduction>10</mechanicalReduction>-->
+<!--		</actuator>-->
+<!--	  </transmission>-->
+<!--	</macro>-->
 </robot>

Commit message: Model Spawn Successful
With ROS Noetic macros to be called as xacro:<macro_name>
mybot.gazebo had a couple of variables missing $ sign which caused a string to be passed to the macro and could not allow the compiler to evaluate a math expression

File: ROSject_2/src/mybot_description/urdf/macros.xacro (robot description, xacro)
@@ -2,7 +2,7 @@
 <robot xmlns:xacro="http://www.ros.org/wiki/xacro"> <!-- NAMESPACE WAS MISSING, USE xacro:macro instead of just macro -->
 	<xacro:macro name="cylinder_inertia" params="m r h">
-	  <inertia  ixx="${m*(3*r*r+h*h)/12}" ixy = "0" ixz = "0"
-		iyy="${m*(3*r*r+h*h)/12}" iyz = "0"
-		izz="${m*r*r/2}"
+	  <inertia  ixx="${m*(3*r*r+h*h)/12.0}" ixy = "0" ixz = "0"
+		iyy="${m*(3*r*r+h*h)/12.0}" iyz = "0"
+		izz="${m*r*r/2.0}"
 	  />
 	</xacro:macro>
@@ -19,51 +19,51 @@
 	  />
 	</xacro:macro>
-<!--	<macro name="wheel" params="lr tY">-->
-<!--	  <link name="${lr}_wheel">-->
-<!--		<collision>-->
-<!--		  <origin xyz="0 0 0" rpy="0 ${PI/2} ${PI/2}" />-->
-<!--		  <geometry>-->
-<!--			<cylinder length="${wheelWidth}" radius="${wheelRadius}"/>-->
-<!--		  </geometry>-->
-<!--		</collision>-->
-<!--		<visual>-->
-<!--		  <origin xyz="0 0 0" rpy="0 ${PI/2} ${PI/2}" />-->
-<!--		  <geometry>-->
-<!--			<cylinder length="${wheelWidth}" radius="${wheelRadius}"/>-->
-<!--		  </geometry>-->
-<!--		  <material name="black"/>-->
-<!--		</visual>-->
-<!--		<inertial>-->
-<!--		  <origin xyz="0 0 0" rpy="0 ${PI/2} ${PI/2}" />-->
-<!--		  <mass value="${wheelMass}"/>-->
-<!--		  <cylinder_inertia m="${wheelMass}" r="${wheelRadius}" h="${wheelWidth}"/>-->
-<!--		</inertial>-->
-<!--	  </link>-->
-<!--	  <gazebo reference="${lr}_wheel">-->
-<!--		<mu1 value="1.0"/>-->
-<!--		<mu2 value="1.0"/>-->
-<!--		<kp  value="10000000.0" />-->
-<!--		<kd  value="1.0" />-->
-<!--		<fdir1 value="1 0 0"/>-->
-<!--		<material>Gazebo/Black</material>-->
-<!--	  </gazebo>-->
-<!--	  <joint name="${lr}_wheel_hinge" type="continuous">-->
-<!--		<parent link="chassis"/>-->
-<!--		<child link="${lr}_wheel"/>-->
-<!--	  <origin xyz="${-wheelPos+chassisLength/2} ${tY*wheelWidth/2+tY*chassisWidth/2} ${wheelRadius}" rpy="0 0 0" />-->
-<!--		<axis xyz="0 1 0" rpy="0 0 0" />-->
-<!--		<limit effort="10000" velocity="10000"/>-->
-<!--		<joint_properties damping="0.0" friction="0.0"/>-->
-<!--	  </joint>-->
-<!--	  <transmission name="${lr}_trans">-->
-<!--		<type>transmission_interface/SimpleTransmission</type>-->
-<!--		<joint name="${lr}_wheel_hinge">-->
-<!--		  <hardwareInterface>EffortJointInterface</hardwareInterface>-->
-<!--		</joint>-->
-<!--		<actuator name="${lr}Motor">-->
-<!--		  <hardwareInterface>EffortJointInterface</hardwareInterface>-->
-<!--		  <mechanicalReduction>10</mechanicalReduction>-->
-<!--		</actuator>-->
-<!--	  </transmission>-->
-<!--	</macro>-->
+	<xacro:macro name="wheel" params="lr tY">
+	  <link name="${lr}_wheel">
+		<collision>
+		  <origin xyz="0 0 0" rpy="0 ${PI/2} ${PI/2}" />
+		  <geometry>
+			<cylinder length="${wheelWidth}" radius="${wheelRadius}"/>
+		  </geometry>
+		</collision>
+		<visual>
+		  <origin xyz="0 0 0" rpy="0 ${PI/2} ${PI/2}" />
+		  <geometry>
+			<cylinder length="${wheelWidth}" radius="${wheelRadius}"/>
+		  </geometry>
+		  <material name="black"/>
+		</visual>
+		<inertial>
+		  <origin xyz="0 0 0" rpy="0 ${PI/2} ${PI/2}" />
+		  <mass value="${wheelMass}"/>
+		  <cylinder_inertia m="${wheelMass}" r="${wheelRadius}" h="${wheelWidth}"/>
+		</inertial>
+	  </link>
+	  <gazebo reference="${lr}_wheel">
+		<mu1 value="1.0"/>
+		<mu2 value="1.0"/>
+		<kp  value="10000000.0" />
+		<kd  value="1.0" />
+		<fdir1 value="1 0 0"/>
+		<material>Gazebo/Black</material>
+	  </gazebo>
+	  <joint name="${lr}_wheel_hinge" type="continuous">
+		<parent link="chassis"/>
+		<child link="${lr}_wheel"/>
+	  <origin xyz="${-wheelPos+chassisLength/2} ${tY*wheelWidth/2+tY*chassisWidth/2} ${wheelRadius}" rpy="0 0 0" />
+		<axis xyz="0 1 0" rpy="0 0 0" />
+		<limit effort="10000" velocity="10000"/>
+		<joint_properties damping="0.0" friction="0.0"/>
+	  </joint>
+	  <transmission name="${lr}_trans">
+		<type>transmission_interface/SimpleTransmission</type>
+		<joint name="${lr}_wheel_hinge">
+		  <hardwareInterface>EffortJointInterface</hardwareInterface>
+		</joint>
+		<actuator name="${lr}Motor">
+		  <hardwareInterface>EffortJointInterface</hardwareInterface>
+		  <mechanicalReduction>10</mechanicalReduction>
+		</actuator>
+	  </transmission>
+	</xacro:macro>
 </robot>

File: ROSject_2/src/mybot_description/urdf/mybot.xacro (robot description, xacro)
@@ -1,33 +1,60 @@
 <?xml version='1.0'?>
 <robot name="mybot" xmlns:xacro="http://www.ros.org/wiki/xacro">
+	<!-- Put here the robot properties common to the model -->
 	<xacro:include filename="$(find mybot_description)/urdf/mybot.gazebo" />
 	<xacro:include filename="$(find mybot_description)/urdf/materials.xacro" />
-<!--	<xacro:include filename="$(find mybot_description)/urdf/macros.xacro" />-->
+	<xacro:include filename="$(find mybot_description)/urdf/macros.xacro" />
+	<xacro:property name="PI" value="3.1415926535897931"/>
+	<xacro:property name="chassisHeight" value="0.1"/>
+	<xacro:property name="chassisLength" value="0.4"/>
+	<xacro:property name="chassisWidth" value="0.2"/>
+	<xacro:property name="chassisMass" value="50.0"/>
+	<xacro:property name="casterRadius" value="0.08"/>
+	<xacro:property name="casterMass" value="5.0"/>
+	<xacro:property name="wheelWidth" value="0.05"/>
+	<xacro:property name="wheelRadius" value="0.1"/>
+	<xacro:property name="wheelPos" value="0.2"/>
+	<xacro:property name="wheelMass" value="5.0"/>
+	<xacro:property name="cameraSize" value="0.05"/>
+	<xacro:property name="cameraMass" value="0.1"/>
+	<!-- End of common prperties description -->
+<!--	<link name="footprint">-->
+<!--	<inertial>-->
+<!--		<inertia name="baseFrameInertia">-->
+<!--			ixx="0.0" ixy="0.0" ixz="0.0"-->
+<!--			iyy="0.0" iyz="0.0"-->
+<!--			izz="0.0"/>-->
+<!--		</inertia>-->
+<!--	</inertial>-->
+<!--	</link>-->
+<!--	<joint name="base_joint" type="fixed">-->
+<!--		<parent link="footprint"/>-->
+<!--		<child link="chassis"/>-->
+<!--	</joint>-->
 	<link name='chassis'>
 		<pose>0 0 0.1 0 0 0</pose>
-		<inertial>
-			<mass value="10.0"/>
-			<origin xyz="0.0 0 0.1" rpy=" 0 0 0"/>
-			<inertia
-					ixx="0.5" ixy="0" ixz="0"
-					iyy="1.0" iyz="0"
-					izz="0.1"
-			/>
-		</inertial>
-		<collision name='collision'>
+<!--		Box of chassis properties-->
+		<collision name="chassisCollision">
+			<origin xyz="0 0 ${wheelRadius}" rpy="0 0 0"/>
 			<geometry>
-				<box size=".4 .2 .1"/>
+				<box size="${chassisLength} ${chassisWidth} ${chassisHeight}"/>
 			</geometry>
 		</collision>
-		<visual name='chassis_visual'>
-			<origin xyz="0 0 0" rpy=" 0 0 0"/>
+		<visual name ="chassisVisual">
+			<origin xyz="0 0 ${wheelRadius}" rpy="0 0 0"/>
 			<geometry>
-				<box size=".4 .2 .1"/>
+				<box size="${chassisLength} ${chassisWidth} ${chassisHeight}"/>
 			</geometry>
+			<material name="orange"/>
 		</visual>
-		<collision name='caster_collision'>
-			<origin xyz="-0.15 0 -0.05" rpy=" 0 0 0"/>
+		<inertial name="chassisInertia">
+			<origin xyz="0 0 ${wheelRadius}" rpy="0 0 0"/>
+			<mass value="${chassisMass}"/>
+			<xacro:box_inertia m="${chassisMass}" x="${chassisLength}" y="${chassisWidth}" z="${chassisHeight}"/>
+		</inertial>
+		<collision name="casterCollision">
+			<origin xyz="-0.2 0 -0.05" rpy=" 0 0 0"/>
 			<geometry>
-				<sphere radius="0.05"/>
+				<sphere radius="${casterRadius}"/>
 			</geometry>
 			<surface>
@@ -42,8 +69,8 @@
 			</surface>
 		</collision>
-		<visual name='caster_visual'>
-			<origin xyz="-0.15 0 -0.05" rpy=" 0 0 0"/>
+		<visual name="casterVisual">
+			<origin xyz="-0.2 0 -0.05" rpy=" 0 0 0"/>
 			<geometry>
-				<sphere radius="0.05"/>
+				<sphere radius="${casterRadius}"/>
 			</geometry>
 		</visual>
@@ -51,48 +78,57 @@
 	<link name="left_wheel">
 		<!--origin xyz="0.1 0.13 0.1" rpy="0 1.5707 1.5707"/-->
-		<collision name="collision">
+		<collision name="collisionLWheel">
 			<origin xyz="0 0 0" rpy="0 1.5707 1.5707"/>
 			<geometry>
-				<cylinder radius="0.1" length="0.05"/>
+				<cylinder radius="${wheelRadius}" length="${wheelWidth}"/>
 			</geometry>
 		</collision>
-		<visual name="left_wheel_visual">
+		<visual name="visualLWheel">
 			<origin xyz="0 0 0" rpy="0 1.5707 1.5707"/>
 			<geometry>
-				<cylinder radius="0.1" length="0.05"/>
+				<cylinder radius="${wheelRadius}" length="${wheelWidth}"/>
 			</geometry>
 		</visual>
 		<inertial>
 			<origin xyz="0 0 0" rpy="0 1.5707 1.5707"/>
-			<mass value="5"/>
-			<cylinder_inertia m="5" r="0.1" h="0.05"/>
-			<inertia
-					ixx="1.0" ixy="0.0" ixz="0.0"
-					iyy="1.0" iyz="0.0"
-					izz="1.0"/>
+			<mass value="${wheelMass}"/>
+			<xacro:cylinder_inertia m="${wheelMass}" r="${wheelRadius}" h="${wheelWidth}"/>
+			<!--			ixx="${wheelMass*(3*wheelRadius*wheelRadius+wheelWidth*wheelWidth)/12}"-->
+<!--			<inertia-->
+<!--					ixx="${wheelMass*(3*wheelRadius*wheelRadius+wheelWidth*wheelWidth)/12}"-->
+<!--					ixy="0.0"-->
+<!--					iyy="${wheelMass*(3*wheelRadius*wheelRadius+wheelWidth*wheelWidth)/12}"-->
+<!--					ixz="0.0"-->
+<!--					izz="wheelMass*wheelRadius*wheelRadius/2.0"-->
+<!--					iyz="0.0"-->
+<!--			/>-->
 		</inertial>
 	</link>
 	<link name="right_wheel">
 		<!--origin xyz="0.1 -0.13 0.1" rpy="0 1.5707 1.5707"/-->
-		<collision name="collision">
+		<collision name="collisionRWheel">
 			<origin xyz="0 0 0" rpy="0 1.5707 1.5707"/>
 			<geometry>
-				<cylinder radius="0.1" length="0.05"/>
+				<cylinder radius="${wheelRadius}" length="${wheelWidth}"/>
 			</geometry>
 		</collision>
-		<visual name="right_wheel_visual">
+		<visual name="visualRWheel">
 			<origin xyz="0 0 0" rpy="0 1.5707 1.5707"/>
 			<geometry>
-				<cylinder radius="0.1" length="0.05"/>
+				<cylinder radius="${wheelRadius}" length="${wheelWidth}"/>
 			</geometry>
 		</visual>
 		<inertial>
 			<origin xyz="0 0 0" rpy="0 1.5707 1.5707"/>
-			<mass value="5"/>
-			<cylinder_inertia m="5" r="0.1" h="0.05"/>
-			<inertia
-					ixx="1.0" ixy="0.0" ixz="0.0"
-					iyy="1.0" iyz="0.0"
-					izz="1.0"/>
+			<mass value="${wheelMass}"/>
+			<xacro:cylinder_inertia m="${wheelMass}" r="${wheelRadius}" h="${wheelWidth}"/>
+<!--		<inertia-->
+<!--				ixx="${wheelMass*(3*wheelRadius*wheelRadius+wheelWidth*wheelWidth)/12}"-->
+<!--				ixy="0.0"-->
+<!--				iyy="${wheelMass*(3*wheelRadius*wheelRadius+wheelWidth*wheelWidth)/12}"-->
+<!--				ixz="0.0"-->
+<!--				izz="wheelMass*wheelRadius*wheelRadius/2.0"-->
+<!--				iyz="0.0"-->
+<!--		/>-->
 		</inertial>
 	</link>

Commit message: Macros for left and right wheel utilized. Model spawn successful. Material spawn still unresolved.Wheels and Caster color spawn successful

File: ROSject_2/src/mybot_description/urdf/macros.xacro (robot description, xacro)
@@ -37,5 +37,5 @@
 		  <origin xyz="0 0 0" rpy="0 ${PI/2} ${PI/2}" />
 		  <mass value="${wheelMass}"/>
-		  <cylinder_inertia m="${wheelMass}" r="${wheelRadius}" h="${wheelWidth}"/>
+		  <xacro:cylinder_inertia m="${wheelMass}" r="${wheelRadius}" h="${wheelWidth}"/>
 		</inertial>
 	  </link>
@@ -59,8 +59,8 @@
 		<type>transmission_interface/SimpleTransmission</type>
 		<joint name="${lr}_wheel_hinge">
-		  <hardwareInterface>EffortJointInterface</hardwareInterface>
+		  <EffortJointInterface>EffortJointInterface</EffortJointInterface>
 		</joint>
 		<actuator name="${lr}Motor">
-		  <hardwareInterface>EffortJointInterface</hardwareInterface>
+		  <EffortJointInterface>EffortJointInterface</EffortJointInterface>
 		  <mechanicalReduction>10</mechanicalReduction>
 		</actuator>

File: ROSject_2/src/mybot_description/urdf/materials.xacro (robot description, xacro)
@@ -13,13 +13,13 @@
 <color rgba="0.2 0.2 0.2 1.0"/>
 </material>
-<material name="orange">
-<color rgba="${255/255} ${108/255} ${10/255} 1.0"/>
-</material>
-<material name="brown">
-<color rgba="${222/255} ${207/255} ${195/255} 1.0"/>
-</material>
-<material name="red">
-<color rgba="0.8 0.0 0.0 1.0"/>
-</material>
+	<material name="orange">
+		<color rgba="0.8 0.4 0.0 1.0"/>
+	</material>
+	<material name="brown">
+		<color rgba="${222/255} ${207/255} ${195/255} 1.0"/>
+	</material>
+	<material name="red">
+		<color rgba="0.8 0.0 0.0 1.0"/>
+	</material>
 <material name="white">
 <color rgba="1.0 1.0 1.0 1.0"/>

File: ROSject_2/src/mybot_description/urdf/mybot.xacro (robot description, xacro)
@@ -10,5 +10,5 @@
 	<xacro:property name="chassisWidth" value="0.2"/>
 	<xacro:property name="chassisMass" value="50.0"/>
-	<xacro:property name="casterRadius" value="0.08"/>
+	<xacro:property name="casterRadius" value="0.1"/>
 	<xacro:property name="casterMass" value="5.0"/>
 	<xacro:property name="wheelWidth" value="0.05"/>
@@ -19,17 +19,17 @@
 	<xacro:property name="cameraMass" value="0.1"/>
 	<!-- End of common prperties description -->
-<!--	<link name="footprint">-->
-<!--	<inertial>-->
-<!--		<inertia name="baseFrameInertia">-->
-<!--			ixx="0.0" ixy="0.0" ixz="0.0"-->
-<!--			iyy="0.0" iyz="0.0"-->
-<!--			izz="0.0"/>-->
-<!--		</inertia>-->
-<!--	</inertial>-->
-<!--	</link>-->
-<!--	<joint name="base_joint" type="fixed">-->
-<!--		<parent link="footprint"/>-->
-<!--		<child link="chassis"/>-->
-<!--	</joint>-->
+	<link name="footprint">
+	<inertial>
+		<inertia name="baseFrameInertia">
+			ixx="0.0" ixy="0.0" ixz="0.0"
+			iyy="0.0" iyz="0.0"
+			izz="0.0"/>
+		</inertia>
+	</inertial>
+	</link>
+	<joint name="base_joint" type="fixed">
+		<parent link="footprint"/>
+		<child link="chassis"/>
+	</joint>
 	<link name='chassis'>
 		<pose>0 0 0.1 0 0 0</pose>
@@ -41,10 +41,10 @@
 			</geometry>
 		</collision>
-		<visual name ="chassisVisual">
+		<visual>
 			<origin xyz="0 0 ${wheelRadius}" rpy="0 0 0"/>
 			<geometry>
 				<box size="${chassisLength} ${chassisWidth} ${chassisHeight}"/>
 			</geometry>
-			<material name="orange"/>
+			<material name="blue"/>
 		</visual>
 		<inertial name="chassisInertia">
@@ -53,99 +53,30 @@
 			<xacro:box_inertia m="${chassisMass}" x="${chassisLength}" y="${chassisWidth}" z="${chassisHeight}"/>
 		</inertial>
-		<collision name="casterCollision">
-			<origin xyz="-0.2 0 -0.05" rpy=" 0 0 0"/>
+	</link>
+	<joint name="fixed" type="fixed">
+		<parent link="chassis"/>
+		<child link="caster_wheel"/>
+	</joint>
+	<link name="caster_wheel">
+		<collision>
+			<origin xyz="${casterRadius-chassisLength/2} 0 ${casterRadius-chassisHeight+wheelRadius}" rpy="0 0 0"/>
 			<geometry>
 				<sphere radius="${casterRadius}"/>
 			</geometry>
-			<surface>
-				<friction>
-					<ode>
-						<mu>0</mu>
-						<mu2>0</mu2>
-						<slip1>1.0</slip1>
-						<slip2>1.0</slip2>
-					</ode>
-				</friction>
-			</surface>
 		</collision>
-		<visual name="casterVisual">
-			<origin xyz="-0.2 0 -0.05" rpy=" 0 0 0"/>
+		<visual>
+			<origin xyz="${casterRadius-chassisLength/2} 0 ${casterRadius-chassisHeight+wheelRadius}" rpy="0 0 0"/>
 			<geometry>
 				<sphere radius="${casterRadius}"/>
 			</geometry>
-		</visual>
-	</link>
-	<link name="left_wheel">
-		<!--origin xyz="0.1 0.13 0.1" rpy="0 1.5707 1.5707"/-->
-		<collision name="collisionLWheel">
-			<origin xyz="0 0 0" rpy="0 1.5707 1.5707"/>
-			<geometry>
-				<cylinder radius="${wheelRadius}" length="${wheelWidth}"/>
-			</geometry>
-		</collision>
-		<visual name="visualLWheel">
-			<origin xyz="0 0 0" rpy="0 1.5707 1.5707"/>
-			<geometry>
-				<cylinder radius="${wheelRadius}" length="${wheelWidth}"/>
-			</geometry>
+			<material name="red"/>
 		</visual>
 		<inertial>
-			<origin xyz="0 0 0" rpy="0 1.5707 1.5707"/>
-			<mass value="${wheelMass}"/>
-			<xacro:cylinder_inertia m="${wheelMass}" r="${wheelRadius}" h="${wheelWidth}"/>
-			<!--			ixx="${wheelMass*(3*wheelRadius*wheelRadius+wheelWidth*wheelWidth)/12}"-->
-<!--			<inertia-->
-<!--					ixx="${wheelMass*(3*wheelRadius*wheelRadius+wheelWidth*wheelWidth)/12}"-->
-<!--					ixy="0.0"-->
-<!--					iyy="${wheelMass*(3*wheelRadius*wheelRadius+wheelWidth*wheelWidth)/12}"-->
-<!--					ixz="0.0"-->
-<!--					izz="wheelMass*wheelRadius*wheelRadius/2.0"-->
-<!--					iyz="0.0"-->
-<!--			/>-->
+			<origin xyz="${casterRadius-chassisLength/2} 0 ${casterRadius-chassisHeight+wheelRadius}" rpy="0 0 0"/>
+			<mass value="${casterMass}"/>
+			<xacro:sphere_inertia m="${casterMass}" r="${casterRadius}"/>
 		</inertial>
 	</link>
-	<link name="right_wheel">
-		<!--origin xyz="0.1 -0.13 0.1" rpy="0 1.5707 1.5707"/-->
-		<collision name="collisionRWheel">
-			<origin xyz="0 0 0" rpy="0 1.5707 1.5707"/>
-			<geometry>
-				<cylinder radius="${wheelRadius}" length="${wheelWidth}"/>
-			</geometry>
-		</collision>
-		<visual name="visualRWheel">
-			<origin xyz="0 0 0" rpy="0 1.5707 1.5707"/>
-			<geometry>
-				<cylinder radius="${wheelRadius}" length="${wheelWidth}"/>
-			</geometry>
-		</visual>
-		<inertial>
-			<origin xyz="0 0 0" rpy="0 1.5707 1.5707"/>
-			<mass value="${wheelMass}"/>
-			<xacro:cylinder_inertia m="${wheelMass}" r="${wheelRadius}" h="${wheelWidth}"/>
-<!--		<inertia-->
-<!--				ixx="${wheelMass*(3*wheelRadius*wheelRadius+wheelWidth*wheelWidth)/12}"-->
-<!--				ixy="0.0"-->
-<!--				iyy="${wheelMass*(3*wheelRadius*wheelRadius+wheelWidth*wheelWidth)/12}"-->
-<!--				ixz="0.0"-->
-<!--				izz="wheelMass*wheelRadius*wheelRadius/2.0"-->
-<!--				iyz="0.0"-->
-<!--		/>-->
-		</inertial>
-	</link>
-	<joint type="continuous" name="left_wheel_hinge">
-		<origin xyz="0.1 0.15 0" rpy="0 0 0"/>
-		<child link="left_wheel"/>
-		<parent link="chassis"/>
-		<axis xyz="0 1 0" rpy="0 0 0"/>
-		<limit effort="100" velocity="100"/>
-		<joint_properties damping="0.0" friction="0.0"/>
-	</joint>
-	<joint type="continuous" name="right_wheel_hinge">
-		<origin xyz="0.1 -0.15 0" rpy="0 0 0"/>
-		<child link="right_wheel"/>
-		<parent link="chassis"/>
-		<axis xyz="0 1 0" rpy="0 0 0"/>
-		<limit effort="100" velocity="100"/>
-		<joint_properties damping="0.0" friction="0.0"/>
-	</joint>
+	<xacro:wheel lr="left" tY="1"/>
+	<xacro:wheel lr="right" tY="-1"/>
 </robot>
