Commit message: Branch initializer commit Trying to resolve issue with ROS Noetic version of transmission hardware interface in left and right wheel hinges

File: ROSject_2/src/mybot_description/urdf/macros.xacro (robot description, xacro)
@@ -59,11 +59,20 @@
 		<type>transmission_interface/SimpleTransmission</type>
 		<joint name="${lr}_wheel_hinge">
-		  <EffortJointInterface>EffortJointInterface</EffortJointInterface>
+		  <hardware_interface>JointStateInterface</hardware_interface>
 		</joint>
 		<actuator name="${lr}Motor">
-		  <EffortJointInterface>EffortJointInterface</EffortJointInterface>
+		  <hardware_interface>JointStateInterface</hardware_interface>
 		  <mechanicalReduction>10</mechanicalReduction>
 		</actuator>
 	  </transmission>
+<!--		  <type>transmission_interface/SimpleTransmission</type>-->
+<!--		  <joint name="${lr}_wheel_hinge">-->
+<!--			  <hardwareInterface>EffortJointInterface</hardwareInterface>-->
+<!--		  </joint>-->
+<!--		  <actuator name="${lr}Motor">-->
+<!--			  <hardwareInterface>EffortJointInterface</hardwareInterface>-->
+<!--			  <mechanicalReduction>10</mechanicalReduction>-->
+<!--		  </actuator>-->
+<!--	  </transmission>-->
 	</xacro:macro>
 </robot>

Commit message: Hardware interface issue resolved Check macros.xacro for reference URL Controller spawn (joint1_position_controller etc) error occured due to controller_spawner receiving joint1_position_controller which is an invalid argument

File: ROSject_2/src/mybot_description/urdf/macros.xacro (robot description, xacro)
@@ -59,8 +59,9 @@
 		<type>transmission_interface/SimpleTransmission</type>
 		<joint name="${lr}_wheel_hinge">
-		  <hardware_interface>JointStateInterface</hardware_interface>
+			<hardwareInterface>hardware_interface/EffortJointInterface</hardwareInterface>
 		</joint>
 		<actuator name="${lr}Motor">
-		  <hardware_interface>JointStateInterface</hardware_interface>
+			<hardwareInterface>hardware_interface/EffortJointInterface</hardwareInterface>
+<!--			https://answers.ros.org/question/372646/controller_manager-not-publishing-joint_state-topic/-->
 		  <mechanicalReduction>10</mechanicalReduction>
 		</actuator>

File: ROSject_2/src/mybot_description/urdf/mybot.xacro (robot description, xacro)
@@ -33,4 +33,5 @@
 <!--		<child link="chassis"/>-->
 <!--	</joint>-->
+<!--	<link name="dummy_link" />-->
 	<link name='chassis'>
 		<pose>0 0 0.1 0 0 0</pose>
@@ -55,4 +56,8 @@
 		</inertial>
 	</link>
+<!--	<joint name="dummy" type="fixed">-->
+<!--		<parent link="dummy_link" />-->
+<!--		<child link="base_link" />-->
+<!--	</joint>-->
 	<joint name="fixed" type="fixed">
 		<parent link="chassis"/>
